File: alt-panel/alt-panel.kicad_pcb (KiCad board)
At the start: 2 copper layers, 50.5 x 128.5 mm, 4 parts

Commit message: Trace corrections, panel corrections
Parts:
- added REF**: LEDisc, diy-nabra:LEDisc, F.Cu at (49.2, 69.1)
- added REF**: Freq, diy-nabra:Freq, F.Cu at (31.5, 92.8)
- added REF**: Cross, diy-nabra:Cross, F.Cu at (31.5, 101.5)
- added REF**: Star, diy-nabra:Star, F.Cu at (19.5, 83.9)
- added REF**: Star, diy-nabra:Star, F.Cu at (19.5, 33.4)
- added REF**: Cross, diy-nabra:Cross, F.Cu at (31.5, 51.0)
- added REF**: Vol, diy-nabra:Vol, F.Cu at (19.5, 109.4)
- added REF**: Vol, diy-nabra:Vol, F.Cu at (19.5, 59.0)
- added REF**: Freq, diy-nabra:Freq, F.Cu at (31.5, 42.3)
Other:
- outline, holes or cut-outs redrawn

Commit message: Panel tweak
Parts:
- moved REF** 0.85 mm to (19.5, 110.2)
- moved REF** 0.75 mm to (19.5, 59.8)
Changed lines of the file:
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@@
   )
   (footprint "diy-nabra:Vol" (layer "F.Cu")
-    (at 19.5 109.4)
+    (at 19.5 110.25)
     (attr through_hole)
     (fp_text reference "REF**" (at 0 -0.5 unlocked) (layer "F.SilkS") hide
@@
       (effects (font (size 1 1) (thickness 0.15)))
     )
-    (fp_line (start 3.7 1.75) (end 3.7 -2.35) (layer "F.SilkS") (width 0.5))
-    (fp_line (start 3.7 -2.35) (end -5 1.75) (layer "F.SilkS") (width 0.5))
-    (fp_line (start -4.9 1.75) (end 3.7 1.75) (layer "F.SilkS") (width 0.5))
+    (fp_line (start 3.5 -2.85) (end -4.5 1.25) (layer "F.SilkS") (width 0.5))
+    (fp_line (start 3.5 1.25) (end 3.5 -2.85) (layer "F.SilkS") (width 0.5))
+    (fp_line (start -4.5 1.25) (end 3.5 1.25) (layer "F.SilkS") (width 0.5))
   )
   (footprint "diy-nabra:Vol" (layer "F.Cu")
-    (at 19.5 59)
+    (at 19.5 59.75)
     (attr through_hole)
     (fp_text reference "REF**" (at 0 -0.5 unlocked) (layer "F.SilkS") hide
@@
       (effects (font (size 1 1) (thickness 0.15)))
     )
-    (fp_line (start 3.7 -2.35) (end -5 1.75) (layer "F.SilkS") (width 0.5))
-    (fp_line (start 3.7 1.75) (end 3.7 -2.35) (layer "F.SilkS") (width 0.5))
-    (fp_line (start -4.9 1.75) (end 3.7 1.75) (layer "F.SilkS") (width 0.5))
+    (fp_line (start 3.5 -2.85) (end -4.5 1.25) (layer "F.SilkS") (width 0.5))
+    (fp_line (start -4.5 1.25) (end 3.5 1.25) (layer "F.SilkS") (width 0.5))
+    (fp_line (start 3.5 1.25) (end 3.5 -2.85) (layer "F.SilkS") (width 0.5))
   )
   (footprint "MountingHole:MountingHole_3.2mm_M3" (layer "F.Cu")
@@
       (effects (font (size 1 1) (thickness 0.15)))
     )
-    (fp_line (start -4 0.0125) (end -1 -2.375) (layer "F.SilkS") (width 0.5))
-    (fp_line (start -1 2.125) (end -4 0.0125) (layer "F.SilkS") (width 0.5))
     (fp_line (start 1 2.125) (end 1 -2.375) (layer "F.SilkS") (width 0.5))
     (fp_line (start 1 -2.375) (end 4 0) (layer "F.SilkS") (width 0.5))
+    (fp_line (start -4 0.0125) (end -1 -2.375) (layer "F.SilkS") (width 0.5))
     (fp_line (start -1 -2.375) (end -1 2.125) (layer "F.SilkS") (width 0.5))
+    (fp_line (start -1 2.125) (end -4 0.0125) (layer "F.SilkS") (width 0.5))
     (fp_line (start 4 0) (end 1 2.125) (layer "F.SilkS") (width 0.5))
   )
@@
       (effects (font (size 1 1) (thickness 0.15)))
     )
+    (fp_line (start 5.5 -2.5) (end 2.5 -2.5) (layer "F.SilkS") (width 0.5))
     (fp_line (start 2.5 -5.5) (end -2.5 -5.5) (layer "F.SilkS") (width 0.5))
+    (fp_line (start -5.5 2.5) (end -2.5 2.5) (layer "F.SilkS") (width 0.5))
+    (fp_line (start 2.5 -2.5) (end 2.5 -5.5) (layer "F.SilkS") (width 0.5))
     (fp_line (start 2.5 5.5) (end 2.5 2.5) (layer "F.SilkS") (width 0.5))
+    (fp_line (start 5.5 -2.5) (end 5.5 2.5) (layer "F.SilkS") (width 0.5))
+    (fp_line (start -5.5 -2.5) (end -5.5 2.5) (layer "F.SilkS") (width 0.5))
+    (fp_line (start -2.5 5.5) (end 2.5 5.5) (layer "F.SilkS") (width 0.5))
     (fp_line (start -2.5 -2.5) (end -5.5 -2.5) (layer "F.SilkS") (width 0.5))
-    (fp_line (start 5.5 -2.5) (end 2.5 -2.5) (layer "F.SilkS") (width 0.5))
     (fp_line (start 2.5 2.5) (end 5.5 2.5) (layer "F.SilkS") (width 0.5))
     (fp_line (start -2.5 2.5) (end -2.5 5.5) (layer "F.SilkS") (width 0.5))
-    (fp_line (start -5.5 2.5) (end -2.5 2.5) (layer "F.SilkS") (width 0.5))
-    (fp_line (start -2.5 5.5) (end 2.5 5.5) (layer "F.SilkS") (width 0.5))
-    (fp_line (start 2.5 -2.5) (end 2.5 -5.5) (layer "F.SilkS") (width 0.5))
-    (fp_line (start -5.5 -2.5) (end -5.5 2.5) (layer "F.SilkS") (width 0.5))
-    (fp_line (start 5.5 -2.5) (end 5.5 2.5) (layer "F.SilkS") (width 0.5))
     (fp_line (start -2.5 -5.5) (end -2.5 -2.5) (layer "F.SilkS") (width 0.5))
   )
@@
   (gr_circle (center 31.5 84) (end 37.5 84) (layer "User.3") (width 0.1) (fill none))
   (dimension (type aligned) (layer "User.1")
+    (pts (xy 51.5 139.25) (xy 51.5 141.25))
+    (height -2.499999)
+    (gr_text "2.0000 mm" (at 52.849999 140.25 90) (layer "User.1")
+      (effects (font (size 1 1) (thickness 0.15)))
+    )
+    (format (units 3) (units_format 1) (precision 4))
+    (style (thickness 0.1) (arrow_length 1.27) (text_position_mode 0) (extension_height 0.58642) (extension_offset 0.5) keep_text_aligned)
+  )
+  (dimension (type aligned) (layer "User.1")
     (pts (xy 17.75 15.75) (xy 12.67 15.75))
     (height 9)
@@
     (style (thickness 0.1) (arrow_length 1.27) (text_position_mode 0) (extension_height 0.58642) (extension_offset 0.5) keep_text_aligned)
   )
+  (group "" (id 27681715-2ba6-4dfd-9a2e-91b6ab9c6a17)
+    (members
+      0dd679fb-3342-4495-8f46-87d90ffb3922
+      17a524e9-2232-4e6c-b234-7909776be5ba
+      191a3ef5-45ae-472c-a381-d5cfc3729146
+      1c09915f-4ecd-4b60-acd9-37a648da8530
+      298b6cf3-7571-40e9-91a8-8d8f607d830c
+      3457bd42-b342-4a7e-9385-d8e5fb766d0e
+      3a34a2ae-1c1a-4c34-bbee-6e07c7739dfa
+      482f6fe6-1d29-4321-902f-8a401a3924a3
+      4ccff719-06f0-485d-962c-fa132c23b4a8
+      587121d6-3236-4003-91fa-3989581afb7a
+      65e2956f-91c2-41a7-afdf-8e7e92a86bf8
+      6745a3ec-1725-41d2-9f08-029c8795c7f5
+      69abaf12-6dc6-4186-bb74-782c2b9c764f
+      6aea4dff-be2e-4e93-a3e1-8933cefab5cf
+      6cc2b798-549c-47c9-8d90-92cef0f224d7
+      6d037aa9-3f18-4a45-a482-4c4d100e9fb8
+      6dd4ab15-5ab6-432d-ba04-64dfca5faa1a
+      6f7a01f3-3429-42c3-80ba-2e07664dd98e
+      72738d5a-a734-4ada-9b0d-84fa63113902
+      73202435-e4f6-444b-8fc0-959909272018
+      788581d7-2bde-4edb-95c9-cc62a47dbe31
+      85bbeac3-50d8-43b7-9f20-abb71dbf451c
+      8ffb6052-8579-4e48-b51f-add2e339496e
+      900d2b26-f4d7-4327-986a-7d98c9ceb27a
+      9d54d75b-3ff0-4f20-ac52-01223b4351de
+      a3a496ef-ecb5-4327-8c96-02074eddf609
+      b0078421-ac0d-41fa-a591-d885f5bcad86
+      b5b34b8f-722e-4c6e-96e3-8b15f514691e
+      c110298a-573d-47d8-ba18-7bb0785721b7
+      c3c1d49a-f915-4f7c-b9fd-e3da4e4eec74
+      c54b70ee-92ce-48d8-9a7b-5086d86ff3f9
+      c5d67f8d-73cc-4282-9296-1d6446eac536
+      d47075a5-eb30-42bf-84ee-dca01c4ed9a5
+      d9cb865c-1eae-47c8-9211-e18811831454
+      e7b9f806-0886-4cab-9e69-1f0ccd2a5c07
+      e86b7121-b6d4-45a2-b0d0-9647ae41abae
+      fc1d0977-be5e-4372-b948-fe4a97ed379b
+    )
+  )
 )
